File: Uno_v1.0.sch (EAGLE design)
At the start: 60 parts, among them CN1 POWER_JACK, CN2 47346-0001, CN3 DIGITAL10, CN4 DIGITAL8, CN5 ICSP, CN6 POWER8, CN7 ANALOG6, IC1 AMS1117-5.0, IC2 AMS1117-3.3, IC3 MCP6002T-I/SN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

Commit message: Add second footprint for atmega328. Move components a little.
Parts:
- added U3: ATMEGA328P-MU, SparkFun-IC-Microcontroller:ATMEGA328P_VQFNVQFN
Connections:
- net 5V: now also U3.AVCC, U3.VCC
- net A0: now also U3.PC0(ADC0)
- net A1: now also U3.PC1(ADC1)
- net A2: now also U3.PC2(ADC2)
- net A3: now also U3.PC3(ADC3)
- net A4_SDA: now also U3.PC4(ADC4/SDA)
- net A5_SCL: now also U3.PC5(ADC5/SCL)
- net AREF: now also U3.AREF
- net D0_RX: now also U3.PD0(RXD)
- net D10_SS: now also U3.PB2(SS/OC1B)
- net D11_MOSI: now also U3.PB3(MOSI/OC2)
- net D12_MISO: now also U3.PB4(MISO)
- net D13_SCK: now also U3.PB5(SCK)
- net D1_TX: now also U3.PD1(TXD)
- net D2: now also U3.PD2(INT0)
- net D3_PWM: now also U3.PD3(INT1)
- net D4: now also U3.PD4(XCK/T0)
- net D5_PWM: now also U3.PD5(T1)
- net D6_PWM: now also U3.PD6(AIN0)
- net D7: now also U3.PD7(AIN1)
- net D8: now also U3.PB0(ICP)
- net D9_PWM: now also U3.PB1(OC1A)
- net GND: now also U3.GND@1, U3.GND@2, U3.GND@PAD
- net MCU_OSC_IN: now also U3.PB6(XTAL1/TOSC1)
- net MCU_OSC_OUT: now also U3.PB7(XTAL2/TOSC2)
- net RESET: now also U3.PC6(/RESET)
Other:
- note added: "Main MCU (extra optional footprint)"
Changed lines of the file:
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@@
 <part name="LOGO2" library="_my_logos" deviceset="MFDECLOGO" device="_L_40MM"/>
 <part name="GND24" library="SparkFun-PowerSymbols" library_urn="urn:adsk.eagle:library:530" deviceset="GND" device=""/>
+<part name="FRAME3" library="frames" library_urn="urn:adsk.eagle:library:229" deviceset="DINA4_L" device=""/>
+<part name="GND25" library="SparkFun-PowerSymbols" library_urn="urn:adsk.eagle:library:530" deviceset="GND" device=""/>
+<part name="SUPPLY5" library="SparkFun-PowerSymbols" library_urn="urn:adsk.eagle:library:530" deviceset="5V" device=""/>
+<part name="U3" library="SparkFun-IC-Microcontroller" library_urn="urn:adsk.eagle:library:525" deviceset="ATMEGA328P_VQFN" device="VQFN" package3d_urn="urn:adsk.eagle:package:38958/1" value="ATMEGA328P-MU"/>
 </parts>
 <sheets>
@@
 </segment>
 </net>
+</nets>
+</sheet>
+<sheet>
+<plain>
+<text x="254" y="7.62" size="2.54" layer="94">1.0</text>
+<text x="165.1" y="27.94" size="2.54" layer="94">(c) Andriy Golovnya</text>
+<text x="198.12" y="7.62" size="2.54" layer="94">20201015-UNO-V1.0</text>
+<text x="101.6" y="132.08" size="2.54" layer="94">Main MCU (extra optional footprint)</text>
+</plain>
+<instances>
+<instance part="FRAME3" gate="G$1" x="0" y="0" smashed="yes"/>
+<instance part="FRAME3" gate="G$2" x="162.56" y="0" smashed="yes">
+<attribute name="LAST_DATE_TIME" x="175.26" y="1.27" size="2.54" layer="94"/>
+<attribute name="SHEET" x="248.92" y="1.27" size="2.54" layer="94"/>
+<attribute name="DRAWING_NAME" x="180.34" y="19.05" size="2.54" layer="94"/>
+</instance>
+<instance part="GND25" gate="1" x="101.6" y="60.96" smashed="yes">
+<attribute name="VALUE" x="99.06" y="58.166" size="1.778" layer="96"/>
+</instance>
+<instance part="SUPPLY5" gate="G$1" x="101.6" y="116.84" smashed="yes">
+<attribute name="VALUE" x="101.6" y="119.634" size="1.778" layer="96"/>
+</instance>
+<instance part="U3" gate="G$1" x="127" y="91.44" smashed="yes">
+<attribute name="NAME" x="109.22" y="125.222" size="1.778" layer="95"/>
+<attribute name="VALUE" x="109.22" y="58.42" size="1.778" layer="96"/>
+</instance>
+</instances>
+<busses>
+</busses>
+<nets>
+<net name="GND" class="3">
+<segment>
+<wire x1="104.14" y1="68.58" x2="101.6" y2="68.58" width="0.1524" layer="91"/>
+<wire x1="101.6" y1="68.58" x2="101.6" y2="66.04" width="0.1524" layer="91"/>
+<wire x1="101.6" y1="66.04" x2="101.6" y2="63.5" width="0.1524" layer="91"/>
+<wire x1="104.14" y1="66.04" x2="101.6" y2="66.04" width="0.1524" layer="91"/>
+<junction x="101.6" y="66.04"/>
+<pinref part="GND25" gate="1" pin="GND"/>
+<pinref part="U3" gate="G$1" pin="GND@1"/>
+<pinref part="U3" gate="G$1" pin="GND@2"/>
+<pinref part="U3" gate="G$1" pin="GND@PAD"/>
+<wire x1="104.14" y1="63.5" x2="101.6" y2="63.5" width="0.1524" layer="91"/>
+<junction x="101.6" y="63.5"/>
+</segment>
+</net>
+<net name="MCU_OSC_IN" class="0">
+<segment>
+<wire x1="104.14" y1="96.52" x2="96.52" y2="96.52" width="0.1524" layer="91"/>
+<label x="88.9" y="96.52" size="1.778" layer="95"/>
+<pinref part="U3" gate="G$1" pin="PB6(XTAL1/TOSC1)"/>
+</segment>
+</net>
+<net name="MCU_OSC_OUT" class="0">
+<segment>
+<wire x1="104.14" y1="91.44" x2="96.52" y2="91.44" width="0.1524" layer="91"/>
+<label x="86.36" y="91.44" size="1.778" layer="95"/>
+<pinref part="U3" gate="G$1" pin="PB7(XTAL2/TOSC2)"/>
+</segment>
+</net>
+<net name="5V" class="3">
+<segment>
+<wire x1="101.6" y1="114.3" x2="101.6" y2="116.84" width="0.1524" layer="91"/>
+<wire x1="101.6" y1="116.84" x2="104.14" y2="116.84" width="0.1524" layer="91"/>
+<wire x1="104.14" y1="114.3" x2="101.6" y2="114.3" width="0.1524" layer="91"/>
+<pinref part="SUPPLY5" gate="G$1" pin="5V"/>
+<junction x="101.6" y="116.84"/>
+<pinref part="U3" gate="G$1" pin="VCC"/>
+<pinref part="U3" gate="G$1" pin="AVCC"/>
+</segment>
+</net>
+<net name="AREF" class="0">
+<segment>
+<wire x1="104.14" y1="106.68" x2="96.52" y2="106.68" width="0.1524" layer="91"/>
+<label x="93.98" y="106.68" size="1.778" layer="95"/>
+<pinref part="U3" gate="G$1" pin="AREF"/>
+</segment>
+</net>
+<net name="A5_SCL" class="0">
+<segment>
+<wire x1="152.4" y1="109.22" x2="160.02" y2="109.22" width="0.1524" layer="91"/>
+<label x="154.94" y="109.22" size="1.778" layer="95"/>
+<pinref part="U3" gate="G$1" pin="PC5(ADC5/SCL)"/>
+</segment>
+</net>
+<net name="A4_SDA" class="0">
+<segment>
+<wire x1="152.4" y1="111.76" x2="160.02" y2="111.76" width="0.1524" layer="91"/>
+<label x="154.94" y="111.76" size="1.778" layer="95"/>
+<pinref part="U3" gate="G$1" pin="PC4(ADC4/SDA)"/>
+</segment>
+</net>
+<net name="A3" class="0">
+<segment>
+<wire x1="152.4" y1="114.3" x2="160.02" y2="114.3" width="0.1524" layer="91"/>
+<label x="157.48" y="114.3" size="1.778" layer="95"/>
+<pinref part="U3" gate="G$1" pin="PC3(ADC3)"/>
+</segment>
+</net>
+<net name="A2" class="0">
+<segment>
+<wire x1="152.4" y1="116.84" x2="160.02" y2="116.84" width="0.1524" layer="91"/>
+<label x="157.48" y="116.84" size="1.778" layer="95"/>
+<pinref part="U3" gate="G$1" pin="PC2(ADC2)"/>
+</segment>
+</net>
+<net name="A1" class="0">
+<segment>
+<wire x1="152.4" y1="119.38" x2="160.02" y2="119.38" width="0.1524" layer="91"/>
+<label x="157.48" y="119.38" size="1.778" layer="95"/>
+<pinref part="U3" gate="G$1" pin="PC1(ADC1)"/>
+</segment>
+</net>
+<net name="A0" class="0">
+<segment>
+<wire x1="152.4" y1="121.92" x2="160.02" y2="121.92" width="0.1524" layer="91"/>
+<label x="157.48" y="121.92" size="1.778" layer="95"/>
+<pinref part="U3" gate="G$1" pin="PC0(ADC0)"/>
+</segment>
+</net>
+<net name="D0_RX" class="0">
+<segment>
+<wire x1="152.4" y1="99.06" x2="160.02" y2="99.06" width="0.1524" layer="91"/>
+<label x="154.94" y="99.06" size="1.778" layer="95"/>
+<pinref part="U3" gate="G$1" pin="PD0(RXD)"/>
+</segment>
+</net>
+<net name="D1_TX" class="0">
+<segment>
+<wire x1="152.4" y1="96.52" x2="160.02" y2="96.52" width="0.1524" layer="91"/>
+<label x="154.94" y="96.52" size="1.778" layer="95"/>
+<pinref part="U3" gate="G$1" pin="PD1(TXD)"/>
+</segment>
+</net>
+<net name="D2" class="0">
+<segment>
+<wire x1="152.4" y1="93.98" x2="160.02" y2="93.98" width="0.1524" layer="91"/>
+<label x="157.48" y="93.98" size="1.778" layer="95"/>
+<pinref part="U3" gate="G$1" pin="PD2(INT0)"/>
+</segment>
+</net>
+<net name="D3_PWM" class="0">
+<segment>
+<wire x1="152.4" y1="91.44" x2="160.02" y2="91.44" width="0.1524" layer="91"/>
+<label x="154.94" y="91.44" size="1.778" layer="95"/>
+<pinref part="U3" gate="G$1" pin="PD3(INT1)"/>
+</segment>
+</net>
+<net name="D4" class="0">
+<segment>
+<wire x1="152.4" y1="88.9" x2="160.02" y2="88.9" width="0.1524" layer="91"/>
+<label x="157.48" y="88.9" size="1.778" layer="95"/>
+<pinref part="U3" gate="G$1" pin="PD4(XCK/T0)"/>
+</segment>
+</net>
+<net name="D5_PWM" class="0">
+<segment>
+<wire x1="152.4" y1="86.36" x2="160.02" y2="86.36" width="0.1524" layer="91"/>
+<label x="154.94" y="86.36" size="1.778" layer="95"/>
+<pinref part="U3" gate="G$1" pin="PD5(T1)"/>
+</segment>
+</net>
+<net name="D6_PWM" class="0">
+<segment>
+<wire x1="152.4" y1="83.82" x2="160.02" y2="83.82" width="0.1524" layer="91"/>
+<label x="154.94" y="83.82" size="1.778" layer="95"/>
+<pinref part="U3" gate="G$1" pin="PD6(AIN0)"/>
+</segment>
+</net>
+<net name="D7" class="0">
+<segment>
+<wire x1="152.4" y1="81.28" x2="160.02" y2="81.28" width="0.1524" layer="91"/>
+<label x="157.48" y="81.28" size="1.778" layer="95"/>
+<pinref part="U3" gate="G$1" pin="PD7(AIN1)"/>
+</segment>
+</net>
+<net name="D8" class="0">
+<segment>
+<wire x1="152.4" y1="76.2" x2="160.02" y2="76.2" width="0.1524" layer="91"/>
+<label x="157.48" y="76.2" size="1.778" layer="95"/>
+<pinref part="U3" gate="G$1" pin="PB0(ICP)"/>
+</segment>
+</net>
+<net name="D9_PWM" class="0">
+<segment>
+<wire x1="152.4" y1="73.66" x2="160.02" y2="73.66" width="0.1524" layer="91"/>
+<label x="154.94" y="73.66" size="1.778" layer="95"/>
+<pinref part="U3" gate="G$1" pin="PB1(OC1A)"/>
+</segment>
+</net>
+<net name="D10_SS" class="0">
+<segment>
+<wire x1="152.4" y1="71.12" x2="160.02" y2="71.12" width="0.1524" layer="91"/>
+<label x="154.94" y="71.12" size="1.778" layer="95"/>
+<pinref part="U3" gate="G$1" pin="PB2(SS/OC1B)"/>
+</segment>
+</net>
+<net name="D11_MOSI" class="0">
+<segment>
+<wire x1="152.4" y1="68.58" x2="160.02" y2="68.58" width="0.1524" layer="91"/>
+<label x="154.94" y="68.58" size="1.778" layer="95"/>
+<pinref part="U3" gate="G$1" pin="PB3(MOSI/OC2)"/>
+</segment>
+</net>
+<net name="D12_MISO" class="0">
+<segment>
+<wire x1="152.4" y1="66.04" x2="160.02" y2="66.04" width="0.1524" layer="91"/>
+<label x="154.94" y="66.04" size="1.778" layer="95"/>
+<pinref part="U3" gate="G$1" pin="PB4(MISO)"/>
+</segment>
+</net>
+<net name="D13_SCK" class="0">
+<segment>
+<wire x1="152.4" y1="63.5" x2="160.02" y2="63.5" width="0.1524" layer="91"/>
+<label x="154.94" y="63.5" size="1.778" layer="95"/>
+<pinref part="U3" gate="G$1" pin="PB5(SCK)"/>
+</segment>
+</net>
+<net name="RESET" class="0">
+<segment>
+<wire x1="104.14" y1="121.92" x2="96.52" y2="121.92" width="0.1524" layer="91"/>
+<label x="93.98" y="121.92" size="1.778" layer="95"/>
+<pinref part="U3" gate="G$1" pin="PC6(/RESET)"/>
+</segment>
+</net>
